Commit message: Add modifications in sim sparus launch to enable simulated profiler

File: data/model/sparus2.urdf (robot description, URDF)
Before this commit: robot Sparus2, 1 links, 0 joints
Links:
- added link seaking_profiler
Joints:
- added joint robot2profiler: type continuous, parent sparus2, child seaking_profiler, origin xyz=0.7 0.0 -0.14 rpy=0 0 3.141592653589793, axis 0 0 1
